Commit message: Changed a few directory issues

File: Gazebo_task_testfiles/test5/robotgame/install/mobile_robot/share/mobile_robot/model/mobile_robot.xacro (robot description, xacro)
@@ -39,5 +39,5 @@
   </link>
   <xacro:wheels/>
-  <!--<xacro:sensors/>
-  <xacro:zed2_camera/>-->
+  <xacro:sensors/>
+  <!--<xacro:zed2_camera/>-->
 </robot>

File: Gazebo_task_testfiles/test5/robotgame/install/mobile_robot/share/mobile_robot/model/sensors.xacro (robot description, xacro)
@@ -4,8 +4,40 @@
   <!-- Lidar Sensor -->
     <link name="lidar_link">
-      <pose>0.0 0.0 0.3 0 0 0</pose>  <!-- Adjusted position -->
       <visual>
         <geometry>
-          <cylinder radius="0.05" length="0.1"/>
+          <cylinder radius="0.07" length="0.05"/>
+        </geometry>
+        <material name="Gazebo/Red">
+          <color rgba="1.0 0.0 0.0 1.0"/>
+        </material>
+      </visual>
+    </link>
+    <joint name="lidar_joint" type="fixed">
+      <parent link="base_link"/>
+      <child link="lidar_link"/>
+      <origin xyz="0 0 ${body_height/2 + 0.025}"/>
+    </joint>
+  <!-- IMU Sensor -->
+    <link name="imu_link">
+      <pose>0.0 0.0 0.0 0 0 0</pose>
+      <visual>
+        <geometry>
+          <box size="0.03 0.03 0.01"/>
+        </geometry>
+        <material name="green">
+          <color rgba="0.0 1.0 0.0 1.0"/>
+        </material>
+      </visual>
+    </link>
+    <joint name="imu_joint" type="fixed">
+      <parent link="base_link"/>
+      <child link="imu_link"/>
+      <origin xyz="0.0 0.0 0.0"/>
+    </joint>
+  <!--    GPS Sensor     -->
+    <link name="pole_link">
+      <visual>
+        <geometry>
+          <cylinder radius="0.01" length="0.4"/>
         </geometry>
         <material name="red">
@@ -13,47 +45,14 @@
         </material>
       </visual>
-      <sensor type="ray" name="lidar">
-        <plugin name="gazebo_ros_laser" filename="libgazebo_ros_ray_sensor.so">
-          <ros>
-            <remapping>scan:=/scan</remapping>
-          </ros>
-        </plugin>
-      </sensor>
     </link>
-    <joint name="lidar_joint" type="fixed">
+    <joint name="pole_joint" type="fixed">
       <parent link="base_link"/>
-      <child link="lidar_link"/>
-      <origin xyz="0.0 0.0 0.3"/>
+      <child link="pole_link"/>
+      <origin xyz="-0.3 0.0 ${body_height/2 + 0.2}"/>
     </joint>
-  <!-- IMU Sensor -->
-    <link name="imu_link">
-      <pose>0.0 0.0 0.15 0 0 0</pose>  <!-- Adjusted position -->
+    <link name="gps_link">
       <visual>
         <geometry>
-          <box size="0.05 0.05 0.02"/>
-        </geometry>
-        <material name="green">
-          <color rgba="0.0 1.0 0.0 1.0"/>
-        </material>
-      </visual>
-      <sensor type="imu" name="imu">
-        <plugin name="gazebo_ros_imu" filename="libgazebo_ros_imu_sensor.so">
-          <ros>
-            <remapping>imu/data:=/imu</remapping>
-          </ros>
-        </plugin>
-      </sensor>
-    </link>
-    <joint name="imu_joint" type="fixed">
-      <parent link="base_link"/>
-      <child link="imu_link"/>
-      <origin xyz="0.0 0.0 0.15"/>
-    </joint>
-  <!-- GPS Sensor -->
-    <link name="gps_link">
-      <pose>-0.15 0.0 0.35 0 0 0</pose>  <!-- Adjusted position -->
-      <visual>
-        <geometry>
-          <sphere radius="0.03"/>
+          <box size="0.05 0.05 0.05"/>
         </geometry>
         <material name="blue">
@@ -61,23 +60,15 @@
         </material>
       </visual>
-      <sensor type="gps" name="gps">
-        <plugin name="gazebo_ros_gps" filename="libgazebo_ros_gps_sensor.so">
-          <ros>
-            <remapping>fix:=/gps</remapping>
-          </ros>
-        </plugin>
-      </sensor>
     </link>
     <joint name="gps_joint" type="fixed">
-      <parent link="base_link"/>
+      <parent link="pole_link"/>
       <child link="gps_link"/>
-      <origin xyz="-0.15 0.0 0.35"/>
+      <origin xyz="0.0 0.0 ${0.2+0.025}"/>
     </joint>
   <!-- Camera Sensor -->
     <link name="camera_link">
-      <pose>0.2 0.0 0.25 0 0 0</pose>  <!-- Adjusted position -->
       <visual>
         <geometry>
-          <box size="0.07 0.03 0.03"/>
+          <box size="0.04 0.05 0.05"/>
         </geometry>
         <material name="gray">
@@ -85,16 +76,9 @@
         </material>
       </visual>
-      <sensor type="camera" name="camera">
-        <plugin name="gazebo_ros_camera" filename="libgazebo_ros_camera.so">
-          <ros>
-            <remapping>image_raw:=/camera/image_raw</remapping>
-          </ros>
-        </plugin>
-      </sensor>
     </link>
     <joint name="camera_joint" type="fixed">
       <parent link="base_link"/>
       <child link="camera_link"/>
-      <origin xyz="0.2 0.0 0.25"/>
+      <origin xyz="${body_length/2+0.04/2} 0.0 0.0"/>
     </joint>
   </xacro:macro>
