Commit message: Finalised the gps task, it's not perfect on correction but it is what it is hehe

File: GPS_task/test2/install/mobile_robot/share/mobile_robot/model/mobile_robot.xacro (robot description, xacro)
@@ -17,6 +17,5 @@
    <link name="base_link">
    	<visual>
-   	<origin xyz="0 0 0" rpy="0 0 0"/>
-   	<geometry>
+   	<origin xyz="0 0 0" rpy="0 0 0"/>   	<geometry>
    		<box size="${body_length} ${body_width} ${body_height}"/>
    	</geometry>
@@ -40,4 +39,5 @@
   <xacro:wheels/>
   <xacro:sensors/>
+  <xacro:zed2_camera/>
   <!--<xacro:zed2_camera/>-->
 </robot>

File: GPS_task/test2/install/mobile_robot/share/mobile_robot/model/sensors.xacro (robot description, xacro)
@@ -64,5 +64,5 @@
       <parent link="pole_link"/>
       <child link="gps_link"/>
-      <origin xyz="0.0 0.0 ${0.2+0.025}"/>
+      <origin xyz="0.0 0.0 ${0.2+0.025}" rpy="0 0 3.14159"/>
     </joint>
   <!-- Camera Sensor -->

File: GPS_task/test2/install/mobile_robot/share/mobile_robot/model/zed2_camera.xacro (robot description, xacro)
@@ -9,6 +9,6 @@
           <box size="0.15 0.05 0.03"/>
         </geometry>
-        <material name="blue">
-          <color rgba="0.0 0.0 1.0 1.0"/>
+        <material name="Yellow">
+          <color rgba="1.0 1.0 0.0 0.7"/>
         </material>
       </visual>
@@ -29,5 +29,5 @@
       <parent link="base_link"/>
       <child link="zed2_link"/>
-      <origin xyz="0.2 0 0.3" rpy="0 0 0"/>  <!-- Adjusted height -->
+      <origin xyz="0.2 0 ${0.15+0.015}" rpy="0 0 1.5708"/>  <!-- Adjusted height -->
     </joint>
     <!-- ZED2 Camera Plugin -->
